Commit message: Added Final Competition Code

File: ros/meam520_labs/urdf/cube.xacro (robot description, xacro)
@@ -63,139 +63,4 @@
       </visual>
     </link>
-    <link name="tag1">
-      <inertial>
-        <mass>0.001</mass>
-        <inertia>
-          <ixx>0.00000000001</ixx>
-          <ixy>0</ixy>
-          <ixz>0</ixz>
-          <iyy>0.00000000001</iyy>
-          <iyz>0</iyz>
-          <izz>0.00000000001</izz>
-        </inertia>
-      </inertial>
-    </link>
-    <link name="tag2">
-      <inertial>
-        <mass>0.001</mass>
-        <inertia>
-          <ixx>0.00000000001</ixx>
-          <ixy>0</ixy>
-          <ixz>0</ixz>
-          <iyy>0.00000000001</iyy>
-          <iyz>0</iyz>
-          <izz>0.00000000001</izz>
-        </inertia>
-      </inertial>
-    </link>
-    <link name="tag3">
-      <inertial>
-        <mass>0.001</mass>
-        <inertia>
-          <ixx>0.00000000001</ixx>
-          <ixy>0</ixy>
-          <ixz>0</ixz>
-          <iyy>0.00000000001</iyy>
-          <iyz>0</iyz>
-          <izz>0.00000000001</izz>
-        </inertia>
-      </inertial>
-    </link>
-    <link name="tag4">
-      <inertial>
-        <mass>0.001</mass>
-        <inertia>
-          <ixx>0.00000000001</ixx>
-          <ixy>0</ixy>
-          <ixz>0</ixz>
-          <iyy>0.00000000001</iyy>
-          <iyz>0</iyz>
-          <izz>0.00000000001</izz>
-        </inertia>
-      </inertial>
-    </link>
-    <link name="tag5">
-      <inertial>
-        <mass>0.001</mass>
-        <inertia>
-          <ixx>0.00000000001</ixx>
-          <ixy>0</ixy>
-          <ixz>0</ixz>
-          <iyy>0.00000000001</iyy>
-          <iyz>0</iyz>
-          <izz>0.00000000001</izz>
-        </inertia>
-      </inertial>
-    </link>
-    <link name="tag6">
-      <inertial>
-        <mass>0.001</mass>
-        <inertia>
-          <ixx>0.00000000001</ixx>
-          <ixy>0</ixy>
-          <ixz>0</ixz>
-          <iyy>0.00000000001</iyy>
-          <iyz>0</iyz>
-          <izz>0.00000000001</izz>
-        </inertia>
-      </inertial>
-      <visual name="marked">
-        <pose>0 0 0.02542 0 0 0</pose>
-        <geometry>
-          <box>
-            <size>0.0508 0.0508 0.0001</size>
-          </box>
-        </geometry>
-        <material>
-          <ambient>.8 .8 .8 1</ambient>
-          <diffuse>.8 .8 .8 1</diffuse>
-          <specular>.8 .8 .8 1</specular>
-          <emissive>0 0 0 0</emissive>
-        </material>
-      </visual>
-    </link>
-    <joint name="tag1_joint" type="fixed">
-      <parent>block</parent>
-      <child>tag1</child>
-      <pose>.0254 0 0 1.5708 0 1.5708</pose>
-      <preserveFixedJoint>true</preserveFixedJoint>
-    </joint>
-    <joint name="tag2_joint" type="fixed">
-      <parent>block</parent>
-      <child>tag2</child>
-      <pose>0 .0254 0 1.5708 0 3.14159</pose>
-      <preserveFixedJoint>true</preserveFixedJoint>
-    </joint>
-    <joint name="tag3_joint" type="fixed">
-      <parent>block</parent>
-      <child>tag3</child>
-      <pose>-.0254 0 0 1.5708 0 -1.5708</pose>
-      <preserveFixedJoint>true</preserveFixedJoint>
-    </joint>
-    <joint name="tag4_joint" type="fixed">
-      <parent>block</parent>
-      <child>tag4</child>
-      <pose>0 -.0254 0 1.5708 0 0</pose>
-      <preserveFixedJoint>true</preserveFixedJoint>
-    </joint>
-    <joint name="tag5_joint" type="fixed">
-      <parent>block</parent>
-      <child>tag5</child>
-      <pose>0 0 -.0254 0 3.14159 -1.5708</pose>
-      <preserveFixedJoint>true</preserveFixedJoint>
-    </joint>
-    <joint name="tag6_joint" type="fixed">
-      <!-- <axis>
-        <xyz>0 0 1</xyz>
-      </axis>
-      <limit>
-        <upper>0</upper>
-        <lower>0</lower>
-      </limit> -->
-      <parent>block</parent>
-      <child>tag6</child>
-      <pose>0 0 .0254 0 0 -1.5708</pose>
-      <preserveFixedJoint>true</preserveFixedJoint>
-    </joint>
   </model>
 </sdf>

File: ros/meam520_labs/urdf/franka_panda.xacro (robot description, xacro)
@@ -4,6 +4,7 @@
 <!-- |    EDITING THIS FILE BY HAND IS NOT RECOMMENDED                                 | -->
 <!-- =================================================================================== -->
-<robot name="panda">
+<robot name="panda" xmlns:xacro="http://www.ros.org/wiki/xacro">
   <!-- If using a different frame with ${connected_to} param, make sure 'world' frame exists in the TF tree -->
+  <xacro:property name="M_PI" value="3.1415926535897931" />
   <joint name="panda_hand_joint" type="fixed">
     <parent link="panda_link8"/>
@@ -217,4 +218,9 @@
     <collision>
       <geometry>
+        <mesh filename="package://franka_panda_description/meshes/collision/link5.stl"/>
+      </geometry>
+    </collision>
+    <!-- <collision>
+      <geometry>
         <mesh filename="package://franka_panda_description/meshes/collision/link5_1.stl"/>
       </geometry>
@@ -229,5 +235,5 @@
         <mesh filename="package://franka_panda_description/meshes/collision/link5_3.stl"/>
       </geometry>
-    </collision>
+    </collision> -->
     <inertial>
       <origin rpy="0 0 0" xyz="-1.1953e-02 4.1065e-02 -3.8437e-02"/>
@@ -297,4 +303,50 @@
     <dynamics damping="1.0" friction="0.5"/>
   </joint>
+ <joint name="camera_joint" type="fixed">
+      <parent link="panda_link7"/>
+      <child link="camera_link"/>
+      <origin rpy="0 ${-pi/2} ${-pi/4 + pi}" xyz="0.03 -0.03  0.1270"/>
+  </joint>
+  <link name="camera_link">
+    <visual>
+        <geometry>
+            <box size="0.02 0.1 0.04" />
+        </geometry>
+    </visual>
+    <collision>
+      <geometry>
+        <box size="0.02 0.1 0.04" />
+      </geometry>
+    </collision>
+  </link>
+  <joint name="camera_optical_joint" type="fixed">
+      <parent link="camera_link"/>
+      <child link="camera_link_optical"/>
+      <origin xyz="0 0 0" rpy="0 0 0"/>
+  </joint>
+  <link name="camera_link_optical"></link>
+  <gazebo reference="camera_link">
+      <material>Gazebo/Black</material>
+      <sensor name="camera" type="camera">
+          <pose> 0 0 0 0 0 0 </pose>
+          <update_rate>30</update_rate>
+          <!-- <visualize>True</visualize> -->
+          <camera>
+              <horizontal_fov>${78 * pi/180.0}</horizontal_fov>
+              <image>
+                  <format>R8G8B8</format>
+                  <width>800</width>
+                  <height>448</height>
+              </image>
+              <clip>
+                  <near>0.1</near>
+                  <far>8.0</far>
+              </clip>
+          </camera>
+          <plugin name="camera_controller" filename="libgazebo_ros_camera.so">
+              <frame_name>camera_link_optical</frame_name>
+          </plugin>
+      </sensor>
+  </gazebo>
   <link name="panda_link8">
     <inertial>
@@ -606,45 +658,34 @@
   </transmission>
   <gazebo reference="panda_link0">
-      <static>true</static>
       <turnGravityOff>true</turnGravityOff>
   </gazebo>
   <gazebo reference="panda_link1">
-      <static>true</static>
       <turnGravityOff>true</turnGravityOff>
   </gazebo>
   <gazebo reference="panda_link2">
-      <static>true</static>
       <turnGravityOff>true</turnGravityOff>
   </gazebo>
   <gazebo reference="panda_link3">
-      <static>true</static>
       <turnGravityOff>true</turnGravityOff>
   </gazebo>
   <gazebo reference="panda_link4">
-      <static>true</static>
       <turnGravityOff>true</turnGravityOff>
   </gazebo>
   <gazebo reference="panda_link5">
-      <static>true</static>
       <turnGravityOff>true</turnGravityOff>
   </gazebo>
   <gazebo reference="panda_link6">
-      <static>true</static>
       <turnGravityOff>true</turnGravityOff>
   </gazebo>
   <gazebo reference="panda_link7">
-      <static>true</static>
       <turnGravityOff>true</turnGravityOff>
   </gazebo>
   <gazebo reference="panda_link8">
-      <static>true</static>
       <turnGravityOff>true</turnGravityOff>
   </gazebo>
   <gazebo reference="panda_leftfinger">
-      <static>true</static>
       <turnGravityOff>true</turnGravityOff>
   </gazebo>
   <gazebo reference="panda_rightfinger">
-      <static>true</static>
       <turnGravityOff>true</turnGravityOff>
   </gazebo>
